File: ABRARACOURCIX_main_board/Input_interface.kicad_sch (KiCad schematic)
At the start: 0 parts

Commit message: Terminé les interconnects
Toutes les interfaces et le power sont terminés. (À vérifier)
Reste à ajouter toutes les connexions au ICM et stm32
Parts:
- added BT_C1: 10uF, Capacitor_SMD:C_0603_1608Metric, symbol Device:C
- added BT_C2: 100nF, Capacitor_SMD:C_0603_1608Metric, symbol Device:C
- added BT_LED1: BLUE, LED_SMD:LED_0603_1608Metric, symbol Device:LED
- added BT_R1: 10k, Resistor_SMD:R_0603_1608Metric, symbol Device:R
- added BT_R2: 1k5, Resistor_SMD:R_0603_1608Metric, symbol Device:R
- added E2: HM-10, ODB:HM-10, symbol ODB_Lib:HM-10
- added J4, J6, J7: Conn_01x04_Socket, symbol Connector:Conn_01x04_Socket
- added J5: Conn_01x05_Socket, Connector_PinHeader_2.54mm:PinHeader_1x05_P2.54mm_Vertical, symbol Connector:Conn_01x05_Socket
- added R3, R4: 10K, symbol Device:R
Connections:
- new net: BT_LED1.2 (A), BT_R2.2
- new net: BT_C2.1, BT_R1.1, E2.11 (RESET)
- new net: BT_R2.1, E2.24 (LED)
- new net: J6.3 (Pin_3), R3.1
- new net +3.3V: J5.3 (Pin_3)
- new net +3V3: BT_C1.1, BT_R1.2, E2.12 (+3.3V)
- new net +5V: J4.1 (Pin_1), J6.1 (Pin_1), J7.1 (Pin_1)
- new net BT_Config/Run: E2.23 (KEY)
- new net GND: BT_C1.2, BT_C2.2, BT_LED1.1 (K), E2.13 (GND), E2.14 (GND__1), E2.21 (GND__2), E2.22 (GND__3), J4.4 (Pin_4), J5.5 (Pin_5), J6.4 (Pin_4), J7.4 (Pin_4), R4.2
- new net HC_RX: J7.2 (Pin_2)
- new net HC_TX: J7.3 (Pin_3)
- new net Luna_RX: J4.2 (Pin_2)
- new net Luna_TX: J4.3 (Pin_3)
- new net SYS_SWCLK: J5.2 (Pin_2)
- new net SYS_SWDIO: J5.1 (Pin_1)
- new net SYS_TRACESWO: J5.4 (Pin_4)
- new net Sonic_Echo: R3.2, R4.1
- new net Sonic_Trig: J6.2 (Pin_2)
- new net UART2_BT_RX: E2.1 (UART_TX)
- new net UART2_BT_TX: E2.2 (UART_RX)
- no-connect marks 0 -> 24
Other:
- note added: "Bluetooth"
- note added: "HC-05 5V pwr/ 3v3 UART"
- note added: "SYS debug (Header pour ST-LINK)"
- note added: "Sensor RX Sensor TX"
- note added: "TF-Luna ToF Single-Point Ranging Solid State LiDAR Sensor (8m, UART / I2C)"
- note added: "Trig: 3-5V output to sensor Echo: 5V logic input to stm32"
- note added: "Ultrasonic sensor 3942 adafruit 5V"

Commit message: Changements obsolete
Connections:
- net UART_CTS: now reaches E2.3 (UART_CTS)
- net UART_RTS: now reaches E2.4 (UART_RTS)
- no-connect marks 24 -> 22
Other:
- note added: "Nécessaire car nos HM-10 sont des clones"
Changed lines of the file:
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@@
+		)
+	)
+	(text "Nécessaire car nos \nHM-10 sont des clones"
+		(exclude_from_sim no)
+		(at 214.63 67.056 0)
+		(effects
+			(font
+				(size 1.27 1.27)
+			)
 		)
 	)
@@
 	)
 	(no_connect
-		(at 170.18 39.37)
-	)
-	(no_connect
 		(at 205.74 57.15)
 	)
@@
 	)
 	(no_connect
-		(at 170.18 41.91)
-	)
-	(no_connect
 		(at 170.18 54.61)
 	)
@@
 	(wire
 		(pts
+			(xy 157.48 41.91) (xy 170.18 41.91)
+		)
+		(stroke
+			(width 0)
+			(type default)
+		)
+	)
+	(wire
+		(pts
 			(xy 167.64 64.77) (xy 170.18 64.77)
 		)
@@
 	(wire
 		(pts
+			(xy 157.48 39.37) (xy 170.18 39.37)
+		)
+		(stroke
+			(width 0)
+			(type default)
+		)
+	)
+	(wire
+		(pts
 			(xy 63.5 41.91) (xy 63.5 40.64)
 		)
@@
 		)
 	)
+	(global_label "UART_CTS"
+		(shape input)
+		(at 157.48 39.37 180)
+		(fields_autoplaced yes)
+		(effects
+			(font
+				(size 1.27 1.27)
+			)
+			(justify right)
+		)
+		(property "Intersheetrefs" "${INTERSHEET_REFS}"
+			(at 145.4234 39.37 0)
+			(effects
+				(font
+					(size 1.27 1.27)
+				)
+				(justify right)
+				(hide yes)
+			)
+		)
+	)
 	(global_label "SYS_TRACESWO"
 		(shape input)
@@
 				(hide yes)
 			)
+		)
+	)
+	(global_label "UART_RTS"
+		(shape input)
+		(at 157.48 41.91 180)
+		(fields_autoplaced yes)
+		(effects
+			(font
+				(size 1.27 1.27)
+			)
+			(justify right)
+		)
+		(property "Intersheetrefs" "${INTERSHEET_REFS}"
+			(at 145.4234 41.91 0)
+			(effects
+				(font
+					(size 1.27 1.27)
+				)
+				(justify right)
+				(hide yes)
+			)
