File: ABRARACOURCIX_main_board/Input_interface.kicad_sch (KiCad schematic)
At the start: 12 parts, among them J4 Conn_01x04_Socket, J5 Conn_01x05_Socket, J6 Conn_01x04_Socket, J7 Conn_01x04_Socket

Commit message: Damn j'ai oublié de push y'a 2 semaines
je sais plus
Changed lines of the file:
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@@
-	(wire
-		(pts
-			(xy 161.29 39.37) (xy 170.18 39.37)
-		)
-		(stroke
-			(width 0)
-			(type default)
-		)
-	)
 	(wire
 		(pts
@@
 		)
 		(stroke
-			(width 0)
-			(type default)
-		)
-	)
-	(wire
-		(pts
-			(xy 161.29 41.91) (xy 170.18 41.91)
-		)
-		(stroke

Commit message: Reprise de contrôle
Schematics terminés
Reste à associer des composantes et vérification
Parts:
- removed BT_C1: 10uF, Capacitor_SMD:C_0603_1608Metric, symbol Device:C
- removed BT_C2: 100nF, Capacitor_SMD:C_0603_1608Metric, symbol Device:C
- removed BT_LED1: BLUE, LED_SMD:LED_0603_1608Metric, symbol Device:LED
- removed BT_R1: 10k, Resistor_SMD:R_0603_1608Metric, symbol Device:R
- removed BT_R2: 1k5, Resistor_SMD:R_0603_1608Metric, symbol Device:R
- removed E2: HM-10, ODB:HM-10, symbol ODB_Lib:HM-10
- removed J7: Conn_01x04_Socket, symbol Connector:Conn_01x04_Socket
- added J4: Conn_01x06_Socket, symbol Connector:Conn_01x06_Socket
- renumbered J4 to #J4, J6 to #J6, R3 to #R3, R4 to #R4
Connections:
- net +5V: now also J4.2 (Pin_2)
- net GND: now also J4.3 (Pin_3)
- net HC_RX: now also J4.5 (Pin_5)
- net HC_TX: now also J4.4 (Pin_4)
- net SYS_TRACESWO renamed NRST
- no-connect marks 22 -> 0
Other:
- note added: "Non utilisé pour la V1"
- note added: "Sensor TX Sensor RX"
- note removed: "Bluetooth"
- note removed: "Nécessaire car nos HM-10 sont des clones"

Commit message: Assignation d<empreintes terminée
Parts:
- J4: footprint (none) -> Connector_PinHeader_2.54mm:PinHeader_1x06_P2.54mm_Horizontal
Changed lines of the file:
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@@
 			)
 		)
-		(property "Footprint" ""
+		(property "Footprint" "Connector_PinHeader_2.54mm:PinHeader_1x06_P2.54mm_Horizontal"
 			(at 53.34 100.33 0)
 			(effects
