File: ABRARACOURCIX_main_board/Input_interface.kicad_sch (KiCad schematic)
At the start: 6 parts, among them J1 Conn_01x05_Socket, J2 Conn_01x06_Socket

Commit message: micro_USB
Parts:
- added C22: 10u, Capacitor_SMD:C_1206_3216Metric_Pad1.33x1.80mm_HandSolder, symbol Device:C
- added J13: microUSB_10118194-0011LF, 10118194-0011LF:AMPHENOL_10118194-0011LF, symbol GAUL_ABRARACOURCIX:microUSB_10118194-0011LF
- added R21, R22, R23: 100k, Resistor_SMD:R_1206_3216Metric_Pad1.30x1.75mm_HandSolder, symbol Device:R
Connections:
- net GND: now also C22.2, J13.5 (GND), J13.S1 (SHIELD), J13.S2 (SHIELD__1), J13.S3 (SHIELD__2), J13.S4 (SHIELD__3), J13.S5 (SHIELD__4), J13.S6 (SHIELD__5), R23.1
- new net: R22.1, R23.2
- new net: J13.1 (VBUS), R21.1
- new net OTG_FS_DM: J13.2 (D-)
- new net OTG_FS_DP: J13.3 (D+)
- new net OTG_FS_ID: J13.4 (ID)
- new net USB_Detect: C22.1, R21.2, R22.2
Other:
- note added: "HC-05 Bluetooth chip 5V pwr/ 3v3 UART"
- note added: "Max 4V sur USB_Detect(USB_OTG_FS)vers pin PA9 Diviseur de tension: 5*200/300 = 3.33 V"
- note added: "Pour lecture de données seulement"
- note removed: "HC-05 5V pwr/ 3v3 UART"
