File: ABRARACOURCIX_main_board/_autosave-Sensors.kicad_sch (KiCad schematic)
At the start: 31 parts, among them U1 STM32F429ZIT6, U2 ICM-42688-P, U5 BNO055, Y1 32.768kHz

Commit message: Avancement
Commencer à relier le stm32
Changed lines of the file:
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@@
-	(wire
-		(pts
-			(xy 223.52 114.3) (xy 223.52 111.76)
-		)
-		(stroke
-			(width 0)
-			(type default)
-		)
-	)
 	(wire
 		(pts
@@
 	(global_label "I2C_SELECT"
 		(shape input)
-		(at 223.52 114.3 180)
+		(at 223.52 111.76 180)
 		(fields_autoplaced yes)
 		(effects
@@
 		)
 		(property "Intersheetrefs" "${INTERSHEET_REFS}"
-			(at 209.7097 114.3 0)
+			(at 209.7097 111.76 0)
 			(effects
 				(font
