File: ABRARACOURCIX_main_board/ABRARACOURCIX_main_board.kicad_pcb (KiCad board)
At the start: 2 copper layers, 140.8 x 111.8 mm, 78 parts, among them J10 Conn_01x03_Socket, J11 Conn_01x03_Socket, J2 XT60PW-M, J3 XT60PW-M, J4 Conn_01x06_Socket, J5 Conn_01x05_Socket, J6 Conn_01x03_Socket, J7 XT60PW-F, J8 Conn_01x03_Socket, J9 Conn_01x03_Socket, K1 Relai_T9GV1L14-5, Q2 NTR4101PT1G, Q3 MMBT3904, U1 STM32F429ZIT6, U2 Current_sens_ACS712ELCTR-20A-T, U3 AZ1117CH-3.3TRG1, U4 Xl4015, U5 BNO055, U6 LMC6482, U7 LMC6482, Y2 ABS07-32.768KHZ-T

Commit message: modifs pas importantes
Parts:
- moved J2 231.5 mm to (366.5, 75.6)
- moved C10 184.8 mm to (278.3, 129.0)
- moved C11 184.8 mm to (278.3, 132.4)
- moved C5 184.8 mm to (278.3, 112.3)
- moved C6 184.8 mm to (278.3, 115.6)
- moved C7 184.8 mm to (278.3, 119.0)
- moved C8 184.8 mm to (278.3, 122.3)
- moved C9 184.8 mm to (278.3, 125.7)
- moved D1 184.8 mm to (310.5, 100.7)
- moved R10 184.8 mm to (296.3, 118.8)
- moved R5 184.8 mm to (296.3, 108.9)
- moved R6 184.8 mm to (296.3, 112.2)
- moved R7 184.8 mm to (296.3, 115.5)
- moved U6 184.8 mm to (303.2, 95.6)
- moved U7 184.8 mm to (303.2, 102.0)
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Other:
- board size 140.8 x 111.8 mm -> 130 x 130 mm
