File: ABRARACOURCIX_main_board/ABRARACOURCIX_main_board.kicad_pcb (KiCad board)
At the start: 2 copper layers, 130 x 130 mm, 79 parts, among them J10 Conn_01x03_Socket, J11 Conn_01x03_Socket, J2 XT60PW-M, J3 XT60PW-M, J4 Conn_01x06_Socket, J5 Conn_01x05_Socket, J6 Conn_01x03_Socket, J7 XT60PW-F, J8 Conn_01x03_Socket, J9 Conn_01x03_Socket, K1 Relai_T9GV1L14-5, Q2 NTR4101PT1G, Q3 MMBT3904, U1 STM32F429ZIT6, U2 Current_sens_ACS712ELCTR-20A-T, U3 AZ1117CH-3.3TRG1, U4 Xl4015, U5 BNO055, U6 LMC6482, U7 LMC6482, U8 STM32F446RETx, Y2 ABS07-32.768KHZ-T

Commit message: Recommencer assignation des composantes
Parts:
- removed BUZ_D2: BAT54T1G, Diode_SMD:D_SOD-123
- removed BUZ_R3: 1k5, Resistor_SMD:R_1206_3216Metric_Pad1.30x1.75mm_HandSolder
- removed C22: 4.7u, Capacitor_SMD:C_1206_3216Metric_Pad1.33x1.80mm_HandSolder
- removed C23: 100nF, Capacitor_SMD:C_1206_3216Metric_Pad1.33x1.80mm_HandSolder
- removed C24: 1uF, Capacitor_SMD:C_1206_3216Metric_Pad1.33x1.80mm_HandSolder
- removed C25, C26: 22pF, Capacitor_SMD:C_1206_3216Metric_Pad1.33x1.80mm_HandSolder
- removed C27: 10u, Capacitor_SMD:C_1206_3216Metric_Pad1.33x1.80mm_HandSolder
- removed C28: 1n, Capacitor_SMD:C_1206_3216Metric_Pad1.33x1.80mm_HandSolder
- removed C29: 0.1u, Capacitor_SMD:C_1206_3216Metric_Pad1.33x1.80mm_HandSolder
- removed C30: 1u, Capacitor_SMD:C_1206_3216Metric_Pad1.33x1.80mm_HandSolder
- removed D3: 599-0410-127F, Diode_SMD:D_1206_3216Metric_Pad1.42x1.75mm_HandSolder
- removed K1: Relai_T9GV1L14-5, Librairie_footprint:Relai_30A_T9GV1L14-5_TEC
- removed PWR_R5: 100k, Resistor_SMD:R_1206_3216Metric_Pad1.30x1.75mm_HandSolder
- removed TP1, TP2, TP3, TP4, TP5: TestPoint, TestPoint:TestPoint_THTPad_2.0x2.0mm_Drill1.0mm
- removed U7: LMC6482, Librairie_footprint:SOIC127P599X175-8N
- removed U8: STM32F446RETx, Package_QFP:LQFP-64_10x10mm_P0.5mm
- removed Y2: ABS07-32.768KHZ-T, Librairie_footprint:XTAL_ABS07-32.768KHZ-T
- added Abraracourcix_moyen: LOGO, Librairie_footprint:Abraracourcix_moyen, F.Cu at (0.00, 37.1)
- added D2: 599-0410-127F, Diode_SMD:D_1206_3216Metric_Pad1.42x1.75mm_HandSolder, F.Cu at (-5.60, 18.7)
- added G***1: LOGO, LOGO, B.Cu at (0.00, 0.00)
- added G***2: LOGO, LOGO, F.Cu at (59.9, -8.40)
- added G***3: LOGO, LOGO, B.Cu at (52.9, 4.70)
- added GND1: TestPoint, TestPoint:TestPoint_THTPad_2.0x2.0mm_Drill1.0mm, F.Cu at (10.4, -36.4)
- added GND2: TestPoint, TestPoint:TestPoint_THTPad_2.0x2.0mm_Drill1.0mm, F.Cu at (15.8, 15.6)
- added J1: Conn_01x05_Socket, Connector_PinHeader_2.54mm:PinHeader_1x05_P2.54mm_Vertical, F.Cu at (36.5, -5.90)
- added J12: Conn_01x02_Pin, Librairie_footprint:MTA_100_2pos, F.Cu at (0.25, -58.0)
- added PWR_R1: 100k, Resistor_SMD:R_1206_3216Metric_Pad1.30x1.75mm_HandSolder, F.Cu at (-21.9, -6.10)
- added Q4: NPN-DSS20201L-7, Package_TO_SOT_SMD:SOT-23, F.Cu at (-26.5, 6.60)
- added Q5: NTR4101PT1G, Package_TO_SOT_SMD:SOT-23-3, F.Cu at (-29.4, -4.95)
- added R17: 10k, Resistor_SMD:R_1206_3216Metric_Pad1.30x1.75mm_HandSolder, F.Cu at (-0.10, -27.8)
- added R18: 30k, Resistor_SMD:R_1206_3216Metric_Pad1.30x1.75mm_HandSolder, F.Cu at (-8.54, -29.9)
- added R19: 40k, Resistor_SMD:R_1206_3216Metric_Pad1.30x1.75mm_HandSolder, F.Cu at (-13.1, -11.3)
- added R20: 10k, Resistor_SMD:R_1206_3216Metric_Pad1.30x1.75mm_HandSolder, F.Cu at (-7.40, -17.8)
- added RX1: TestPoint, TestPoint:TestPoint_THTPad_2.0x2.0mm_Drill1.0mm, F.Cu at (24.9, 7.45)
- added SCL1: TestPoint, TestPoint:TestPoint_THTPad_2.0x2.0mm_Drill1.0mm, F.Cu at (11.1, -25.8)
- added SDA1: TestPoint, TestPoint:TestPoint_THTPad_2.0x2.0mm_Drill1.0mm, F.Cu at (6.20, -25.8)
- added TX1: TestPoint, TestPoint:TestPoint_THTPad_2.0x2.0mm_Drill1.0mm, F.Cu at (24.9, 11.6)
- added Y1: ABS07-32.768KHZ-T, Librairie_footprint:XTAL_ABS07-32.768KHZ-T, F.Cu at (-0.80, -5.60)
- C1: value 22u -> 100n; footprint Resistor_SMD:R_0805_2012Metric -> Capacitor_SMD:C_1206_3216Metric_Pad1.33x1.80mm_HandSolder
- C10, C4: value 100n -> 1u
- C11: value 100n -> 10u; footprint Capacitor_SMD:C_1206_3216Metric_Pad1.33x1.80mm_HandSolder -> Librairie_footprint:CAP_MU_15750_RUB-L
- C12: value 100n -> 100nF
- C13: value 100n -> 1uF
- C14, C15: value 100n -> 22pF
- C16: value 100n -> 0.1u
- C17: value 100n -> 1n
- C18: value 100n -> 10u
- C19: value 4.7u -> 22u
- C2: value 22u -> 100n
- C20: value 4.7u -> 1u
- C21: value 4.7u -> 22u; footprint Capacitor_SMD:C_1206_3216Metric_Pad1.33x1.80mm_HandSolder -> Resistor_SMD:R_0805_2012Metric
- C3: value 10u -> 100n
- C7: value 100n -> 4.7u
- C8, C9: value 100n -> 2.2u
- J10: value Conn_01x03_Socket -> XT60PW-M; footprint Connector_PinHeader_2.54mm:PinHeader_1x03_P2.54mm_Horizontal -> Librairie_footprint:AMASS_XT60PW-M
- J11: value Conn_01x03_Socket -> Conn_01x02_Pin; footprint Connector_PinHeader_2.54mm:PinHeader_1x03_P2.54mm_Horizontal -> Librairie_footprint:MTA_100_2pos
- J2: value XT60PW-M -> Conn_01x06_Socket; footprint Connector_AMASS:AMASS_XT60-F_1x02_P7.20mm_Vertical -> Connector_PinHeader_2.54mm:PinHeader_1x06_P2.54mm_Horizontal
- J3: value XT60PW-M -> Conn_01x03_Socket; footprint Librairie_footprint:AMASS_XT60PW-M -> Connector_PinHeader_2.54mm:PinHeader_1x03_P2.54mm_Horizontal
- J4: value Conn_01x06_Socket -> Conn_01x03_Socket; footprint Connector_PinHeader_2.54mm:PinHeader_1x06_P2.54mm_Horizontal -> Connector_PinHeader_2.54mm:PinHeader_1x03_P2.54mm_Horizontal
- J5: value Conn_01x05_Socket -> Conn_01x03_Socket; footprint Connector_PinHeader_2.54mm:PinHeader_1x05_P2.54mm_Vertical -> Connector_PinHeader_2.54mm:PinHeader_1x03_P2.54mm_Horizontal
- J7: value XT60PW-F -> Conn_01x03_Socket; footprint Librairie_footprint:AMASS_XT60PW-F -> Connector_PinHeader_2.54mm:PinHeader_1x03_P2.54mm_Horizontal
- J8: value Conn_01x03_Socket -> XT60PW-M; footprint Connector_PinHeader_2.54mm:PinHeader_1x03_P2.54mm_Horizontal -> Connector_AMASS:AMASS_XT60-F_1x02_P7.20mm_Vertical
- J9: value Conn_01x03_Socket -> XT60PW-F; footprint Connector_PinHeader_2.54mm:PinHeader_1x03_P2.54mm_Horizontal -> Librairie_footprint:AMASS_XT60PW-F
- Q2: value NTR4101PT1G -> DSS20200L-7-PNP
- Q3: value MMBT3904 -> IKD15N60R; footprint Package_TO_SOT_SMD:SOT-23-3 -> Package_TO_SOT_SMD:TO-252-2
- R10: value 3K -> 1k5
- R11, R14: value 30k -> 10k
- R12: value 10k -> 30k
- R15: value 10k -> 40
- R2: value 40 -> 10K
- R3: value 10k -> 10K
- R4: value 20k -> 1K
- R5: value 3K -> 1k
- R6: value 10K -> 10k
- R7: value 10K -> 1k5
- R8: value 40k -> 10k
- R9: value 10k -> 20k
- U1: value STM32F429ZIT6 -> STM32F429VITx; footprint Librairie_footprint:QFP50P2200X2200X160-144N -> Package_QFP:LQFP-100_14x14mm_P0.5mm
- U2: value Current_sens_ACS712ELCTR-20A-T -> BNO055; footprint Librairie_footprint:Current_sens_SOIC127P600X175-8N -> Librairie_footprint:BNO055_LGA28R50P4X10_380X520X100
- U3: value AZ1117CH-3.3TRG1 -> Current_sens_ACS712ELCTR-20A-T; footprint Librairie_footprint:AZ1117CH_3_3TRG1-L -> Librairie_footprint:Current_sens_SOIC127P600X175-8N
- U4: value Xl4015 -> AZ1117CH-3.3TRG1; footprint Librairie_footprint:Buck_breakout_Xl4015 -> Librairie_footprint:AZ1117CH_3_3TRG1-L
- U5: value BNO055 -> LMC6482AIMX/NOPB; footprint Librairie_footprint:BNO055_LGA28R50P4X10_380X520X100 -> Librairie_footprint:SOIC127P599X175-8N
- U6: value LMC6482 -> LMC6482AIMX/NOPB
- moved J10 474.8 mm to (-60.0, -9.25)
- moved J9 471.4 mm to (-60.0, 3.15)
- moved U3 456.9 mm to (-46.5, 0.60)
- moved J8 450.4 mm to (-38.5, -9.20), turned to 180 degrees
- moved Q3 447.6 mm to (-45.1, 9.53), turned to 180 degrees
- moved R2 440.7 mm to (-10.7, 3.10), turned to 90 degrees
- moved J11 439.7 mm to (-21.9, -10.7)
- moved Q2 435.2 mm to (-32.9, 6.80), turned to -90 degrees
- moved J5 435.0 mm to (-12.2, -56.0), turned to 90 degrees
- moved R11 431.3 mm to (-32.9, 12.0)
- moved R14 423.6 mm to (-10.3, -35.6), turned to -90 degrees
- moved DZ1 422.6 mm to (-29.2, -9.15)
- moved R12 416.8 mm to (-6.38, -35.5), turned to 90 degrees
- moved R16 416.2 mm to (0.26, -39.0), turned to 180 degrees
- moved J7 414.9 mm to (12.2, 56.0), turned to -90 degrees
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Connections:
- C1 pad 1: +5V -> +3.3V
- C11 pad 1: +3.3V -> +5V
- C12 pad 1: +3.3V -> GND
- C12 pad 2: GND -> +3.3V
- C13 pad 1: +3.3V -> GND
- C13 pad 2: GND -> Net-(U2-CAP)
- C14 pad 1: +3.3V -> XIN32
- C15 pad 1: +3.3V -> GND
- C15 pad 2: GND -> XOUT32
- C16 pad 1: +3.3V -> +5V
- C17 pad 1: +3.3V -> Net-(U3-FILTER)
- C18 pad 1: +3.3V -> VBAT_sense
- C19 pad 1: GND -> +3.3V
- C19 pad 2: +3.3V -> GND
- C2 pad 1: +3.3V -> GND
- C2 pad 2: GND -> Net-(U1-VREF+)
- C20 pad 1: GND -> Net-(U6B-+)
- C20 pad 2: +3.3V -> GND
- C21 pad 1: GND -> +5V
- C21 pad 2: +3.3V -> GND
- C3 pad 1: VBAT_sense -> +3.3V
- C4 pad 1: +3.3V -> GND
- C4 pad 2: GND -> Net-(U1-VREF+)
- C8 pad 1: +3.3V -> Net-(U1-VCAP_1)
- C8 pad 2: GND -> +3.3V
- C9 pad 1: +3.3V -> Net-(U1-VCAP_1)
- C9 pad 2: GND -> +3.3V
- J10 pad 1: PWM_Servo_1 -> /Power/16V_pre-switch
- J10 pad 2: +5V -> GND
- J11 pad 1: PWM_Servo_4 -> VBAT_sense
- J11 pad 2: +5V -> GND
- J2 pad 1: Net-(J2-+) -> unconnected-(J2-Pin_1-Pad1)
- J2 pad 2: Net-(J2--) -> HC_RX
- J3 pad 1: Net-(J2--) -> PWM_Servo_4
- J3 pad 2: GND -> +5V
- J4 pad 1: unconnected-(J4-Pin_1-Pad1) -> PWM_Servo_3
- J5 pad 1: SYS_SWDIO -> PWM_Servo_2
- J5 pad 2: SYS_SWCLK -> +5V
- J5 pad 3: +3.3V -> GND
- J6 pad 1: PWM_Moteur -> PWM_Servo_1
- J6 pad 2: unconnected-(J6-Pin_2-Pad2) -> +5V
- J7 pad 1: GND -> PWM_Moteur
- J7 pad 2: VBAT -> unconnected-(J7-Pin_2-Pad2)
- J8 pad 1: PWM_Servo_2 -> /Power/16V_post-switch
- J8 pad 2: +5V -> /Power/16V_pre-switch
- J9 pad 1: PWM_Servo_3 -> /Power/GND_IGBT
- J9 pad 2: +5V -> /Power/16V_motor
- R1 pad 1: +3.3V -> Net-(U1-PC1)
- R10 pad 1: +3.3V -> Net-(Q4-PadB)
- R10 pad 2: SDA -> Motor_switch
- R11 pad 1: Net-(U7A--) -> Net-(Q2-PadC)
- R11 pad 2: VBAT_ADC -> GND
- R12 pad 1: Net-(U6B--) -> Net-(U6A--)
- R12 pad 2: Net-(U7A--) -> VBAT_ADC
- R13 pad 1: Net-(U7B--) -> +3.3V
- R13 pad 2: Net-(U7A-+) -> Net-(U5B-+)
- R14 pad 1: GND -> Net-(U5B--)
- R14 pad 2: Net-(U7A-+) -> Net-(U6A--)
- R15 pad 2: Net-(U6B-+) -> Net-(D2-A)
- R16 pad 1: Net-(U6B-+) -> Net-(U5B-+)
- R2 pad 1: Net-(U1A-PC1/ETH_MDC/EVENTOUT) -> +3.3V
- R2 pad 2: Net-(D3-A) -> BNO_RESET
- R3 pad 1: Net-(U2-VIOUT) -> +3.3V
- R3 pad 2: VIout_sense -> BNO_BOOT
- R4 pad 1: VIout_sense -> +3.3V
- R4 pad 2: GND -> SDA
- R6 pad 1: +3.3V -> /Power/GND_IGBT
- R6 pad 2: BNO_BOOT -> Net-(Q4-PadC)
- R7 pad 1: +3.3V -> Net-(Q2-PadB)
- R7 pad 2: BNO_RESET -> Net-(Q4-PadC)
- R8 pad 1: VBAT_sense -> Net-(U3-VIOUT)
- R8 pad 2: Net-(U7B-+) -> VIout_sense
- R9 pad 1: Net-(U7B-+) -> VIout_sense
- U1 pad 10: unconnected-(U1B-PF0/I2C2_SDA/FMC_A0/EVENTOUT-Pad10) -> GND
- U1 pad 100: unconnected-(U1A-PA8/MCO1/TIM1_CH1/I2C3_SCL/USART1_CK/OTG_FS_SOF/LCD_R6/EVENTOUT-Pad100) -> +3.3V
- U1 pad 11: unconnected-(U1B-PF1/I2C2_SCL/FMC_A1/EVENTOUT-Pad11) -> +3.3V
- U1 pad 14: unconnected-(U1B-PF4/FMC_A4/EVENTOUT/ADC3_IN14-Pad14) -> NRST
- U1 pad 16: GND -> Net-(U1-PC1)
- U1 pad 17: +3.3V -> unconnected-(U1-PC2-Pad17)
- U1 pad 19: unconnected-(U1B-PF7/TIM11_CH1/SPI5_SCK/SAI1_MCLK_B/UART7_TX/FMC_NREG/EVENTOUT-Pad19) -> +3.3V
- U1 pad 20: unconnected-(U1B-PF8/SPI5_MISO/SAI1_SCK_B/TIM13_CH1/FMC_NIOWR/EVENTOUT-Pad20) -> GND
- U1 pad 21: unconnected-(U1B-PF9/SPI5_MOSI/SAI1_FS_B/TIM14_CH1/FMC_CD/EVENTOUT-Pad21) -> Net-(U1-VREF+)
- U1 pad 22: unconnected-(U1B-PF10/FMC_INTR/DCMI_D11/LCD_DE/EVENTOUT-Pad22) -> +3.3V
- U1 pad 25: NRST -> unconnected-(U1-PA2-Pad25)
- U1 pad 26: BT_Config/Run -> Motor_switch
- U1 pad 27: Net-(U1A-PC1/ETH_MDC/EVENTOUT) -> GND
- U1 pad 28: unconnected-(U1A-PC2/SPI2_MISO/I2S2EXT_SD/OTG_HS_ULPI_DIR/ETH_MII_TXD2/FMC_SDNE0/EVENTOUT-Pad28) -> +3.3V
- U1 pad 30: +3.3V -> unconnected-(U1-PA5-Pad30)
- U1 pad 31: GND -> unconnected-(U1-PA6-Pad31)
- U1 pad 33: +3.3V -> unconnected-(U1-PC4-Pad33)
- U1 pad 35: unconnected-(U1A-PA1/TIM2_CH2/TIM5_CH2/USART2_RTS/UART4_RX/ETH_MII_RX_CLK/ETH_RMII_REF_CLK/EVENTOUT-Pad35) -> VIout_sense
- U1 pad 36: unconnected-(U1A-PA2/TIM2_CH3/TIM5_CH3/TIM9_CH1/USART2_TX/ETH_MDIO/EVENTOUT-Pad36) -> VBAT_ADC
- U1 pad 37: Motor_switch -> unconnected-(U1-PB2-Pad37)
- U1 pad 38: GND -> unconnected-(U1-PE7-Pad38)
- U1 pad 39: +3.3V -> unconnected-(U1-PE8-Pad39)
- U1 pad 46: VIout_sense -> unconnected-(U1-PE15-Pad46)
- U1 pad 47: VBAT_ADC -> unconnected-(U1-PB10-Pad47)
- U1 pad 49: unconnected-(U1B-PF11/SPI5_MOSI/FMC_SDNRAS/DCMI_D12/EVENTOUT-Pad49) -> Net-(U1-VCAP_1)
- U1 pad 50: unconnected-(U1B-PF12/FMC_A6/EVENTOUT-Pad50) -> +3.3V
- U1 pad 51: GND -> unconnected-(U1-PB12-Pad51)
- U1 pad 52: +3.3V -> unconnected-(U1-PB13-Pad52)
- U1 pad 59: unconnected-(U1B-PE8/TIM1_CH1N/UART7_TX/FMC_D5/EVENTOUT-Pad59) -> PWM_Servo_1
- U1 pad 60: unconnected-(U1B-PE9/TIM1_CH1/FMC_D6/EVENTOUT-Pad60) -> PWM_Servo_2
- U1 pad 61: GND -> PWM_Servo_3
- U1 pad 62: +3.3V -> PWM_Servo_4
- U1 pad 72: +3.3V -> SYS_SWDIO
- U1 pad 73: unconnected-(U1A-PB12/TIM1_BKIN/I2C2_SMBA/SPI2_NSS/I2S2_WS/USART3_CK/CAN2_RX/OTG_HS_ULPI_D5/ETH_MII_TXD0/ETH_RMII_TXD0/OTG_HS_ID/EVENTOUT-Pad73) -> Net-(U1-VCAP_1)
- U1 pad 74: unconnected-(U1A-PB13/TIM1_CH1N/SPI2_SCK/I2S2_CK/USART3_CTS/CAN2_TX/OTG_HS_ULPI_D6/ETH_MII_TXD1/ETH_RMII_TXD1/EVENTOUT-Pad74) -> GND
- U1 pad 75: unconnected-(U1A-PB14/TIM1_CH2N/TIM8_CH2N/SPI2_MISO/I2S2EXT_SD/USART3_RTS/TIM12_CH1/OTG_HS_DM/EVENTOUT-Pad75) -> +3.3V
- U1 pad 76: unconnected-(U1A-PB15/RTC_REFIN/TIM1_CH3N/TIM8_CH3N/SPI2_MOSI/I2S2_SD/TIM12_CH2/OTG_HS_DP/EVENTOUT-Pad76) -> SYS_SWCLK
- U1 pad 81: PWM_Servo_1 -> unconnected-(U1-PD0-Pad81)
- U1 pad 82: PWM_Servo_2 -> unconnected-(U1-PD1-Pad82)
- U1 pad 83: GND -> unconnected-(U1-PD2-Pad83)
- U1 pad 84: +3.3V -> unconnected-(U1-PD3-Pad84)
- U1 pad 85: PWM_Servo_3 -> unconnected-(U1-PD4-Pad85)
- U1 pad 86: PWM_Servo_4 -> HC_RX
- U1 pad 87: unconnected-(U1B-PG2/FMC_A12/EVENTOUT-Pad87) -> HC_TX
- U1 pad 90: unconnected-(U1B-PG5/FMC_A15/FMC_BA1/EVENTOUT-Pad90) -> PWM_Moteur
- U1 pad 91: unconnected-(U1B-PG6/FMC_INT2/DCMI_D12/LCD_R7/EVENTOUT-Pad91) -> BNO_RESET
- U1 pad 92: unconnected-(U1B-PG7/USART6_CK/FMC_INT3/DCMI_D13/LCD_CLK/EVENTOUT-Pad92) -> SCL
- U1 pad 93: unconnected-(U1B-PG8/SPI6_NSS/USART6_RTS/ETH_PPS_OUT/FMC_SDCLK/EVENTOUT-Pad93) -> SDA
- U1 pad 94: GND -> unconnected-(U1-BOOT0-Pad94)
- U1 pad 95: +3.3V -> BNO_BOOT
- U1 pad 96: unconnected-(U1A-PC6/TIM3_CH1/TIM8_CH1/I2S2_MCK/USART6_TX/SDIO_D6/DCMI_D0/LCD_HSYNC/EVENTOUT-Pad96) -> BNO_INT_OUT
- U1 pad 99: unconnected-(U1A-PC9/MCO2/TIM3_CH4/TIM8_CH4/I2C3_SDA/I2S_CKIN/SDIO_D1/DCMI_D3/EVENTOUT-Pad99) -> GND
- U2 pad 1: Net-(J2-+) -> (no net)
- U2 pad 2: Net-(J2-+) -> GND
- U2 pad 3: Net-(Q2-D) -> +3.3V
- U2 pad 4: Net-(Q2-D) -> BNO_BOOT
- U2 pad 6: Net-(U2-FILTER) -> GND
- U2 pad 7: Net-(U2-VIOUT) -> (no net)
- U2 pad 8: +5V -> (no net)
- U3 pad 1: GND -> /Power/16V_post-switch
- U3 pad 2: +3.3V -> /Power/16V_post-switch
- U3 pad 3: VBAT_sense -> /Power/16V_motor
- U3 pad 4: unconnected-(U3-EPAD-Pad4) -> /Power/16V_motor
- U4 pad 1: VBAT_sense -> GND
- U4 pad 2: GND -> +3.3V
- U4 pad 3: +5V -> VBAT_sense
- U4 pad 4: GND -> unconnected-(U4-EPAD-Pad4)
- U5 pad 1: (no net) -> unconnected-(U5-Pad1)
- U5 pad 2: GND -> unconnected-(U5A---Pad2)
- U5 pad 3: +3.3V -> unconnected-(U5A-+-Pad3)
- U5 pad 4: BNO_BOOT -> GND
- U5 pad 5: GND -> Net-(U5B-+)
- U5 pad 6: GND -> Net-(U5B--)
- U5 pad 7: (no net) -> Net-(U5B--)
- U5 pad 8: (no net) -> +3.3V
- U6 pad 1: unconnected-(U6-Pad1) -> VBAT_ADC
- U6 pad 2: unconnected-(U6A---Pad2) -> Net-(U6A--)
- U6 pad 3: unconnected-(U6A-+-Pad3) -> Net-(U6A-+)
Routing:
- net GND: track 0.00 -> 111.6 mm, vias 0 -> 43
- net Net-(U3-VIOUT): track 0.00 -> 77.4 mm, vias 0 -> 6
- net PWM_Servo_4: track 0.00 -> 76.5 mm, vias 0 -> 5
- net PWM_Servo_1: track 0.00 -> 73.1 mm, vias 0 -> 5
- net PWM_Moteur: track 0.00 -> 71.4 mm, vias 0 -> 7
- net PWM_Servo_2: track 0.00 -> 60.9 mm, vias 0 -> 3
- net Motor_switch: track 0.00 -> 53.4 mm, vias 0 -> 6
- net PWM_Servo_3: track 0.00 -> 49.5 mm, vias 0 -> 1
- net VBAT_ADC: track 0.00 -> 49.5 mm, vias 0 -> 2
- net VBAT_sense: track 0.00 -> 42.2 mm, vias 0 -> 2
- net HC_TX: track 0.00 -> 39.4 mm, vias 0 -> 1
- net HC_RX: track 0.00 -> 36.6 mm, vias 0 -> 1
- net SYS_SWCLK: track 0.00 -> 36.0 mm, vias 0 -> 1
- net NRST: track 0.00 -> 35.5 mm, vias 0 -> 1
- net SCL: track 0.00 -> 33.1 mm, vias 0 -> 3
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- added copper zone on F.Cu, net +3.3V
- added copper zone on B.Cu, net +5V
- added copper zone on F.Cu, net +5V
- added copper zone on B.Cu, net /Power/16V_motor
- added copper zone on F.Cu, net /Power/16V_motor
- added copper zone on F.Cu, net /Power/16V_post-switch
- added copper zone on F.Cu, net /Power/16V_pre-switch
- added copper zone on F.Cu, net /Power/GND_IGBT
- added copper zone on B.Cu, net GND
- added copper zone on F.Cu, net GND
Other:
- board size 130 x 130 mm -> 140 x 140 mm
- board text added: "16.8V"
- board text added: "16.8V Moteur"
- board text added: "3v3 Power"
- board text added: "5V"
- board text added: "5V GND"
- board text added: "Abraracourcix le GAULois"
- board text added: "Battery Input"
- board text added: "Battery Input XT60 Mâle"
- board text added: "Debug"
- board text added: "GND"
- board text added: "GND 5V"
- board text added: "GND IGBT"
- board text added: "HC-05 Breakout"
- board text added: "Input 16v8 max"
- board text added: "MTA Buck 5V In"
- board text added: "Output XT60 Female"
- board text added: "Output to ESC"
- board text added: "PWM 5V GND"
- board text added: "PWM Moteur GND"
- board text added: "Projet ABRARACOURCIX V1 GAULxDesign IV 2025 Nathan Armishaw Etienne Bernier Marc-André Tremblay Rémi Plante Félix Dion"
- board text added: "Projet ABRARACOURCIX: Asservissement en Boucles et Régulation Avancée RApide pour le Contrôle d'Objet Unirotorisé Réactifs avec Capteur Inertiel eXpérimental"
- board text added: "RX"
- board text added: "SCL"
- board text added: "SDA"
- board text added: "SWDIO SWCLK 3v3 NRST GND"
- board text added: "TX"
- board text added: "To ON/OFF switch"
