File: ABRARACOURCIX_main_board/ABRARACOURCIX_main_board.kicad_sch (KiCad schematic)
At the start: 17 parts, among them U1 STM32F429VITx

Commit message: Circuit+début PCB
Parts:
- removed C1, C2, C3, C5, C6: 100n, Capacitor_SMD:C_1206_3216Metric_Pad1.33x1.80mm_HandSolder, symbol Device:C
- removed C10, C4: 1u, Capacitor_SMD:C_1206_3216Metric_Pad1.33x1.80mm_HandSolder, symbol Device:C
- removed C7: 4.7u, Capacitor_SMD:C_1206_3216Metric_Pad1.33x1.80mm_HandSolder, symbol Device:C
- removed C8, C9: 2.2u, Capacitor_SMD:C_1206_3216Metric_Pad1.33x1.80mm_HandSolder, symbol Device:C
- removed D1: 599-0410-127F, Diode_SMD:D_1206_3216Metric_Pad1.42x1.75mm_HandSolder, symbol Device:LED
- removed GND1, GND2, RX1, TX1: TestPoint, TestPoint:TestPoint_THTPad_2.0x2.0mm_Drill1.0mm, symbol Connector:TestPoint
- removed R1: 40.2, Resistor_SMD:R_1206_3216Metric_Pad1.30x1.75mm_HandSolder, symbol Device:R
- removed U1: STM32F429VITx, Package_QFP:LQFP-100_14x14mm_P0.5mm, symbol MCU_ST_STM32F4:STM32F429VITx
- added J2: Conn_01x06_Socket, Connector_PinHeader_2.54mm:PinHeader_1x06_P2.54mm_Horizontal, symbol Connector:Conn_01x06_Socket
- added J3, J4, J5, J6, J7: Conn_01x03_Socket, Connector_PinHeader_2.54mm:PinHeader_1x03_P2.54mm_Horizontal, symbol Connector:Conn_01x03_Socket
- added R4: 1K, Resistor_THT:R_Axial_DIN0207_L6.3mm_D2.5mm_P10.16mm_Horizontal, symbol Device:R
- added R5: 1k, Resistor_THT:R_Axial_DIN0207_L6.3mm_D2.5mm_P10.16mm_Horizontal, symbol Device:R
- added U1: STM32F429I-DISC1, Librairie_footprint:MODULE_STM32F429I-DISC1, symbol GAUL_ABRARACOURCIX:STM32F429I-DISC1
- added U2: BNO055_breakout, Librairie_footprint:MODULE_2472, symbol GAUL_ABRARACOURCIX:BNO055_breakout
Connections:
- net +3.3V: now also R4.1, R5.2, U1.P2_1 (3V), U1.P2_2 (3V)
- net GND: now also J2.3 (Pin_3), J3.3 (Pin_3), J4.3 (Pin_3), J5.3 (Pin_3), J6.3 (Pin_3), J7.3 (Pin_3), U1.JP1_1 (GND_1), U1.JP1_2 (GND_1), U1.JP2_1 (GND_2), U1.JP2_2 (GND_2), U1.P1_63 (GND_1), U1.P1_64 (GND_1), U1.P2_11 (GND_2), U1.P2_29 (GND_2), U1.P2_63 (GND_2), U1.P2_64 (GND_2), U2.3 (GND), U2.7 (ADR)
- net HC_RX: now also J2.5 (Pin_5), U1.P1_37 (PD5)
- net HC_TX: now also J2.4 (Pin_4), U1.P1_36 (PD6)
- net PWM_Moteur: now also J7.1 (Pin_1), U1.P1_25 (PB4)
- net PWM_Servo_1: now also J6.1 (Pin_1), U1.P2_58 (PD12)
- net PWM_Servo_2: now also J5.1 (Pin_1), U1.P2_57 (PD13)
- net PWM_Servo_3: now also J4.1 (Pin_1), U1.P2_60 (PD14)
- net PWM_Servo_4: now also J3.1 (Pin_1), U1.P2_59 (PD15)
- net SCL: now also R5.1, U1.P1_23 (PB6), U2.5 (SCL)
- net SDA: now also R4.2, U1.P1_24 (PB7), U2.4 (SDA)
- new net +5V: J2.2 (Pin_2), J3.2 (Pin_2), J4.2 (Pin_2), J5.2 (Pin_2), J6.2 (Pin_2), U1.P1_1 (5V), U1.P1_2 (5V), U1.P1_22 (VDD), U2.1 (VIN)
- new net BNO_Int: U1.P1_20 (PB9), U2.8 (INT)
- new net BNO_Reset: U1.P1_26 (PB5), U2.6 (RST)
- no-connect marks 65 -> 111
Other:
- removed sheet Input_interface
- removed sheet Output_interface
- removed sheet Sensors
- note added: "Blanc Noir"
- note added: "HC-05 5V pwr/ 3v3 UART"
- note added: "Motor IO"
- note added: "PWM - Yellow VCC - Red GND - Brown"
- note added: "Sensor TX Sensor RX"
- note removed: "Inversion RX/TX au MCU"
- note removed: "LED rouge Debug VLED = 2.1V à 30 mA R= (3.3-2.1)/30mA = 40 Ohm"
- note removed: "VDD-VSS"
- note removed: "VDDA-VSSA"
- note removed: "VREF-VSS"

Commit message: PCB terminé
Parts:
- removed R4: 1K, Resistor_THT:R_Axial_DIN0207_L6.3mm_D2.5mm_P10.16mm_Horizontal, symbol Device:R
- removed R5: 1k, Resistor_THT:R_Axial_DIN0207_L6.3mm_D2.5mm_P10.16mm_Horizontal, symbol Device:R
Connections:
- net +3.3V: no longer names the net of U1.P2_1 (3V)
- net +3.3V: no longer U1.P2_2 (3V)
- no-connect marks 111 -> 113
Other:
- moved on the sheet: J7, U2
