File: ABRARACOURCIX_main_board/Power.kicad_sch (KiCad schematic)
At the start: 5 parts, among them J10 XT60PW-M, J8 XT60PW-M, J9 XT60PW-F

Commit message: PCB terminé
Connections:
- net +5V: now also U3.3 (Out+); no longer U3. (Out-)
- net 16V_post-switch: now also U3.1 (In+); no longer U3. (Out-)
- net GND: now also U3.2 (In-), U3.4 (Out-); no longer U3. (Out-)
Changed lines of the file:
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@@
 			)
 		)
-		(pin ""
+		(pin "1"
 		)
-		(pin ""
+		(pin "3"
 		)
-		(pin ""
+		(pin "4"
 		)
-		(pin ""
+		(pin "2"
 		)
 		(instances
