File: ABRARACOURCIX_main_board/Output_interface.kicad_sch (KiCad schematic)
At the start: 11 parts, among them J3 Conn_01x03_Socket, J4 Conn_01x03_Socket, J5 Conn_01x03_Socket, J6 Conn_01x03_Socket, J7 Conn_01x03_Socket, Q1 MMBT3904

Commit message: micro_USB
Parts:
- J7: now not fitted; now left out of the parts list
