File: ABRARACOURCIX_main_board-2025-11-06_181406/ABRARACOURCIX_main_board.kicad_sch (KiCad schematic)
At the start: 6 parts, among them U1 STM32F429ZIT6

Commit message: Modifs au circuit d'alim
Parts:
- removed D3: 599-0410-127F, Diode_SMD:D_1206_3216Metric_Pad1.42x1.75mm_HandSolder, symbol Device:LED
- removed R2: 40, Resistor_SMD:R_1206_3216Metric_Pad1.30x1.75mm_HandSolder, symbol Device:R
- removed TP1, TP2, TP3: TestPoint, TestPoint:TestPoint_THTPad_2.0x2.0mm_Drill1.0mm, symbol Connector:TestPoint
- removed U1: STM32F429ZIT6, Librairie_footprint:QFP50P2200X2200X160-144N, symbol GAUL_ABRARACOURCIX:STM32F429ZIT6
- added C10, C11: 2.2u, Capacitor_SMD:C_1206_3216Metric_Pad1.33x1.80mm_HandSolder, symbol Device:C
- added C12, C14, C4, C5, C6, C7, C8, C9: 100n, Capacitor_SMD:C_1206_3216Metric_Pad1.33x1.80mm_HandSolder, symbol Device:C
- added C13, C15: 1u, Capacitor_SMD:C_1206_3216Metric_Pad1.33x1.80mm_HandSolder, symbol Device:C
- added C19: 4.7u, Capacitor_SMD:C_1206_3216Metric_Pad1.33x1.80mm_HandSolder, symbol Device:C
- added D2: 599-0410-127F, Diode_SMD:D_1206_3216Metric_Pad1.42x1.75mm_HandSolder, symbol Device:LED
- added R17: 40, Resistor_SMD:R_1206_3216Metric_Pad1.30x1.75mm_HandSolder, symbol Device:R
- added TP6, TP7: TestPoint, TestPoint:TestPoint_THTPad_2.0x2.0mm_Drill1.0mm, symbol Connector:TestPoint
- added U9: STM32F429VETx, Package_QFP:LQFP-100_14x14mm_P0.5mm, symbol MCU_ST_STM32F4:STM32F429VETx
Connections:
- net BNO_BOOT: now also U9.95 (PB8)
- net BNO_INT_OUT: now also U9.96 (PB9)
- net BNO_RESET: now also U9.91 (PB5)
- net GND: now also C12.2, C13.2, C14.1, C15.1, C19.2, C4.2, C5.2, C6.2, C7.2, C8.2, C9.2, D2.1 (K), U9.10 (VSS), U9.20 (VSSA), U9.27 (VSS), U9.74 (VSS), U9.99 (VSS)
- net HC_RX: now also TP6.1, U9.86 (PD5)
- net HC_TX: now also TP7.1, U9.87 (PD6)
- net Motor_switch: now also U9.26 (PA3)
- net NRST: now also U9.14 (NRST)
- net PWM_Moteur: now also U9.90 (PB4)
- net PWM_Servo_1: now also U9.59 (PD12)
- net PWM_Servo_2: now also U9.60 (PD13)
- net PWM_Servo_3: now also U9.61 (PD14)
- net PWM_Servo_4: now also U9.62 (PD15)
- net SCL: now also U9.92 (PB6)
- net SDA: now also U9.93 (PB7)
- net SYS_SWCLK: now also U9.76 (PA14)
- net SYS_SWDIO: now also U9.72 (PA13)
- net VBAT_ADC: now also U9.36 (PB1)
- net VIout_sense: now also U9.35 (PB0)
- new net: C10.1, C11.1, U9.49 (VCAP_1), U9.73 (VCAP_2)
- new net: D2.2 (A), R17.2
- new net: R17.1, U9.16 (PC1)
- new net: C14.2, C15.2, U9.21 (VREF+)
- new net +3.3V: C10.2, C11.2, C12.1, C13.1, C19.1, C4.1, C5.1, C6.1, C7.1, C8.1, C9.1, U9.100 (VDD), U9.11 (VDD), U9.19 (VDD), U9.22 (VDDA), U9.28 (VDD), U9.50 (VDD), U9.6 (VBAT), U9.75 (VDD)
- no-connect marks 2 -> 65
Other:
- note added: "VDD-VSS"
- note added: "VDDA-VSSA"
- note added: "VREF-VSS"

Commit message: Placement des composantes 95%
Parts:
- removed C12, C8, C9: 100n, Capacitor_SMD:C_1206_3216Metric_Pad1.33x1.80mm_HandSolder, symbol Device:C
- removed U9: STM32F429VETx, Package_QFP:LQFP-100_14x14mm_P0.5mm, symbol MCU_ST_STM32F4:STM32F429VETx
- added U1: STM32F429VITx, Package_QFP:LQFP-100_14x14mm_P0.5mm, symbol MCU_ST_STM32F4:STM32F429VITx
Connections:
- net +3.3V: now also U1.100 (VDD), U1.11 (VDD), U1.19 (VDD), U1.22 (VDDA), U1.28 (VDD), U1.50 (VDD), U1.6 (VBAT), U1.75 (VDD)
- net BNO_BOOT: now also U1.95 (PB8)
- net BNO_INT_OUT: now also U1.96 (PB9)
- net BNO_RESET: now also U1.91 (PB5)
- net GND: now also U1.10 (VSS), U1.20 (VSSA), U1.27 (VSS), U1.74 (VSS), U1.99 (VSS)
- net HC_RX: now also U1.86 (PD5)
- net HC_TX: now also U1.87 (PD6)
- net Motor_switch: now also U1.26 (PA3)
- net NRST: now also U1.14 (NRST)
- net PWM_Moteur: now also U1.90 (PB4)
- net PWM_Servo_1: now also U1.59 (PD12)
- net PWM_Servo_2: now also U1.60 (PD13)
- net PWM_Servo_3: now also U1.61 (PD14)
- net PWM_Servo_4: now also U1.62 (PD15)
- net SCL: now also U1.92 (PB6)
- net SDA: now also U1.93 (PB7)
- net SYS_SWCLK: now also U1.76 (PA14)
- net SYS_SWDIO: now also U1.72 (PA13)
- net VBAT_ADC: now also U1.36 (PB1)
- net VIout_sense: now also U1.35 (PB0)
- net at C10.1, C11.1: now also U1.49 (VCAP_1), U1.73 (VCAP_2)
- net at R17.1: now also U1.16 (PC1)
- net at C14.2, C15.2: now also U1.21 (VREF+)
Other:
- moved on the sheet: C19

Commit message: Documentation de composantes
Parts:
- added GND1, GND2: TestPoint, TestPoint:TestPoint_THTPad_2.0x2.0mm_Drill1.0mm, symbol Connector:TestPoint
- renumbered TP6 to RX1, TP7 to TX1
Connections:
- net GND: now also GND1.1, GND2.1
Other:
- moved on the sheet: RX1

Commit message: Routing terminé (v1)
Parts:
- renumbered C4 to C1, C13 to C10, C14 to C2, C6 to C3, C15 to C4, C7 to C6, C19 to C7, C11 to C8, C10 to C9, D2 to D1, R17 to R1
Changed lines of the file:
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@@
 		(dnp no)
 		(fields_autoplaced yes)
-		(property "Reference" "C10"
+		(property "Reference" "C9"
 			(at 46.99 143.5101 0)
 			(effects
@@
 			(project ""
 				(path "/0de7b960-2097-47c8-970c-7acab0ada146"
-					(reference "C10")
+					(reference "C9")
 					(unit 1)
 				)
@@
 		(dnp no)
 		(fields_autoplaced yes)
-		(property "Reference" "#PWR064"
+		(property "Reference" "#PWR08"
 			(at 130.81 148.59 0)
 			(effects
@@
 			(project "ABRARACOURCIX_main_board"
 				(path "/0de7b960-2097-47c8-970c-7acab0ada146"
-					(reference "#PWR064")
+					(reference "#PWR08")
 					(unit 1)
 				)
@@
 		(dnp no)
 		(fields_autoplaced yes)
-		(property "Reference" "D2"
+		(property "Reference" "D1"
 			(at 134.62 137.4774 90)
 			(effects
@@
 			(project "ABRARACOURCIX_main_board"
 				(path "/0de7b960-2097-47c8-970c-7acab0ada146"
-					(reference "D2")
+					(reference "D1")
 					(unit 1)
 				)
@@
 		(dnp no)
 		(fields_autoplaced yes)
-		(property "Reference" "#PWR062"
+		(property "Reference" "#PWR05"
 			(at 39.37 97.79 0)
 			(effects
@@
 			(project "ABRARACOURCIX_main_board"
 				(path "/0de7b960-2097-47c8-970c-7acab0ada146"
-					(reference "#PWR062")
+					(reference "#PWR05")
 					(unit 1)
 				)
@@
 		(dnp no)
 		(fields_autoplaced yes)
-		(property "Reference" "R17"
+		(property "Reference" "R1"
 			(at 133.35 128.2699 0)
 			(effects
@@
 			(project "ABRARACOURCIX_main_board"
 				(path "/0de7b960-2097-47c8-970c-7acab0ada146"
-					(reference "R17")
+					(reference "R1")
 					(unit 1)
 				)
@@
 		(dnp no)
 		(fields_autoplaced yes)
-		(property "Reference" "#PWR032"
+		(property "Reference" "#PWR01"
 			(at 90.17 29.21 0)
 			(effects
@@
 			(project "ABRARACOURCIX_main_board"
 				(path "/0de7b960-2097-47c8-970c-7acab0ada146"
-					(reference "#PWR032")
+					(reference "#PWR01")
 					(unit 1)
 				)
@@
 		(dnp no)
 		(fields_autoplaced yes)
-		(property "Reference" "C7"
+		(property "Reference" "C6"
 			(at 187.96 62.23 90)
 			(effects
@@
 			(project "ABRARACOURCIX_main_board"
 				(path "/0de7b960-2097-47c8-970c-7acab0ada146"
-					(reference "C7")
+					(reference "C6")
 					(unit 1)
 				)
@@
 		(dnp no)
 		(fields_autoplaced yes)
-		(property "Reference" "#PWR031"
+		(property "Reference" "#PWR02"
 			(at 181.61 39.37 0)
 			(effects
@@
 			(project "ABRARACOURCIX_main_board"
 				(path "/0de7b960-2097-47c8-970c-7acab0ada146"
-					(reference "#PWR031")
+					(reference "#PWR02")
 					(unit 1)
 				)
@@
 		(dnp no)
 		(fields_autoplaced yes)
-		(property "Reference" "#PWR065"
+		(property "Reference" "#PWR010"
 			(at 97.79 179.07 0)
 			(effects
@@
 			(project "ABRARACOURCIX_main_board"
 				(path "/0de7b960-2097-47c8-970c-7acab0ada146"
-					(reference "#PWR065")
+					(reference "#PWR010")
 					(unit 1)
 				)
@@
 		(dnp no)
 		(fields_autoplaced yes)
-		(property "Reference" "C19"
+		(property "Reference" "C7"
 			(at 187.96 74.93 90)
 			(effects
@@
 			(project "ABRARACOURCIX_main_board"
 				(path "/0de7b960-2097-47c8-970c-7acab0ada146"
-					(reference "C19")
+					(reference "C7")
 					(unit 1)
 				)
@@
 		(dnp no)
 		(fields_autoplaced yes)
-		(property "Reference" "C13"
+		(property "Reference" "C10"
 			(at 187.96 137.16 90)
 			(effects
@@
 			(project "ABRARACOURCIX_main_board"
 				(path "/0de7b960-2097-47c8-970c-7acab0ada146"
-					(reference "C13")
+					(reference "C10")
 					(unit 1)
 				)
@@
 		(dnp no)
 		(fields_autoplaced yes)
-		(property "Reference" "#PWR067"
+		(property "Reference" "#PWR03"
 			(at 46.99 64.77 0)
 			(effects
@@
 			(project "ABRARACOURCIX_main_board"
 				(path "/0de7b960-2097-47c8-970c-7acab0ada146"
-					(reference "#PWR067")
+					(reference "#PWR03")
 					(unit 1)
 				)
@@
 		(on_board yes)
 		(dnp no)
-		(property "Reference" "C11"
+		(property "Reference" "C8"
 			(at 33.02 143.5101 0)
 			(effects
@@
 			(project "ABRARACOURCIX_main_board"
 				(path "/0de7b960-2097-47c8-970c-7acab0ada146"
-					(reference "C11")
+					(reference "C8")
 					(unit 1)
 				)
@@
 		(dnp no)
 		(fields_autoplaced yes)
-		(property "Reference" "C4"
+		(property "Reference" "C1"
 			(at 187.96 27.94 90)
 			(effects
@@
 			(project "ABRARACOURCIX_main_board"
 				(path "/0de7b960-2097-47c8-970c-7acab0ada146"
-					(reference "C4")
+					(reference "C1")
 					(unit 1)
 				)
@@
 		(dnp no)
 		(fields_autoplaced yes)
-		(property "Reference" "C6"
+		(property "Reference" "C3"
 			(at 187.96 39.37 90)
 			(effects
@@
 			(project "ABRARACOURCIX_main_board"
 				(path "/0de7b960-2097-47c8-970c-7acab0ada146"
-					(reference "C6")
+					(reference "C3")
 					(unit 1)
 				)
@@
 		(dnp no)
 		(fields_autoplaced yes)
-		(property "Reference" "#PWR033"
+		(property "Reference" "#PWR04"
 			(at 191.77 92.71 0)
 			(effects
@@
 			(project "ABRARACOURCIX_main_board"
 				(path "/0de7b960-2097-47c8-970c-7acab0ada146"
-					(reference "#PWR033")
+					(reference "#PWR04")
 					(unit 1)
 				)
@@
 		(dnp no)
 		(fields_autoplaced yes)
-		(property "Reference" "C15"
+		(property "Reference" "C4"
 			(at 50.8 50.8 90)
 			(effects
@@
 			(project "ABRARACOURCIX_main_board"
 				(path "/0de7b960-2097-47c8-970c-7acab0ada146"
-					(reference "C15")
+					(reference "C4")
 					(unit 1)
 				)
@@
 		(dnp no)
 		(fields_autoplaced yes)
-		(property "Reference" "#PWR034"
+		(property "Reference" "#PWR06"
 			(at 184.15 135.89 0)
 			(effects
@@
 			(project "ABRARACOURCIX_main_board"
 				(path "/0de7b960-2097-47c8-970c-7acab0ada146"
-					(reference "#PWR034")
+					(reference "#PWR06")
 					(unit 1)
 				)
@@
 		(dnp no)
 		(fields_autoplaced yes)
-		(property "Reference" "#PWR035"
+		(property "Reference" "#PWR09"
 			(at 191.77 151.13 0)
 			(effects
@@
 			(project "ABRARACOURCIX_main_board"
 				(path "/0de7b960-2097-47c8-970c-7acab0ada146"
-					(reference "#PWR035")
+					(reference "#PWR09")
 					(unit 1)
 				)
@@
 		(dnp no)
 		(fields_autoplaced yes)
-		(property "Reference" "C14"
+		(property "Reference" "C2"
 			(at 50.8 39.37 90)
 			(effects
@@
 			(project "ABRARACOURCIX_main_board"
 				(path "/0de7b960-2097-47c8-970c-7acab0ada146"
-					(reference "C14")
+					(reference "C2")
 					(unit 1)
 				)
@@
 		(dnp no)
 		(fields_autoplaced yes)
-		(property "Reference" "#PWR047"
+		(property "Reference" "#PWR07"
 			(at 36.83 142.24 0)
 			(effects
@@
 			(project "ABRARACOURCIX_main_board"
 				(path "/0de7b960-2097-47c8-970c-7acab0ada146"
-					(reference "#PWR047")
-					(unit 1)
-				)
+					(reference "#PWR07")
+					(unit 1)
+				)
