File: ABRARACOURCIX_main_board-2025-11-06_181406/Input_interface.kicad_sch (KiCad schematic)
At the start: 6 parts, among them J4 Conn_01x06_Socket, J5 Conn_01x05_Socket

Commit message: Placement des composantes 95%
Connections:
- no-connect marks 0 -> 2
Changed lines of the file:
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@@
 		(color 0 0 0 0)
+	)
+	(no_connect
+		(at 58.42 95.25)
+	)
+	(no_connect
+		(at 58.42 107.95)
 	)
 	(wire

Commit message: Documentation de composantes
Connections:
- net +5V: now also J4.5 (Pin_5); no longer J4.2 (Pin_2)
- net GND: now also J4.4 (Pin_4); no longer J4.3 (Pin_3)
- net HC_RX: now also J4.2 (Pin_2); no longer J4.5 (Pin_5)
- net HC_TX: now also J4.3 (Pin_3); no longer J4.4 (Pin_4)
Other:
- moved on the sheet: J4
Changed lines of the file:
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@@
 	(symbol
 		(lib_id "Connector:Conn_01x06_Socket")
-		(at 53.34 100.33 0)
-		(mirror y)
+		(at 53.34 102.87 180)
 		(unit 1)
 		(exclude_from_sim no)
@@
 		(dnp no)
 		(property "Reference" "J4"
-			(at 52.07 96.774 0)
+			(at 52.07 106.426 0)
 			(effects
 				(font
@@
 		)
 		(property "Value" "Conn_01x06_Socket"
-			(at 52.578 94.488 0)
+			(at 52.578 108.712 0)
 			(effects
 				(font
@@
 		)
 		(property "Footprint" "Connector_PinHeader_2.54mm:PinHeader_1x06_P2.54mm_Horizontal"
-			(at 53.34 100.33 0)
+			(at 53.34 102.87 0)
 			(effects
 				(font
@@
 		)
 		(property "Datasheet" "~"
-			(at 53.34 100.33 0)
+			(at 53.34 102.87 0)
 			(effects
 				(font
@@
 		)
 		(property "Description" "Generic connector, single row, 01x06, script generated"
-			(at 53.34 100.33 0)
+			(at 53.34 102.87 0)
 			(effects
 				(font
@@
 		)
 		(instances
-			(project ""
+			(project "ABRARACOURCIX_main_board"
 				(path "/0de7b960-2097-47c8-970c-7acab0ada146/6c5d3f5c-4c22-4772-8235-2f35636af7f3"
 					(reference "J4")

Commit message: Routing terminé (v1)
Parts:
- renumbered #J4 to #J1, #J6 to #J2, #R3 to #R1, #R4 to #R2, J5 to J1, J4 to J2
Changed lines of the file:
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@@
 		(dnp no)
 		(fields_autoplaced yes)
-		(property "Reference" "#PWR021"
+		(property "Reference" "#PWR019"
 			(at 69.85 161.29 0)
 			(effects
@@
 			(project "ABRARACOURCIX_main_board"
 				(path "/0de7b960-2097-47c8-970c-7acab0ada146/6c5d3f5c-4c22-4772-8235-2f35636af7f3"
-					(reference "#PWR021")
+					(reference "#PWR019")
 					(unit 1)
 				)
@@
 		(dnp no)
 		(fields_autoplaced yes)
-		(property "Reference" "#PWR016"
+		(property "Reference" "#PWR013"
 			(at 71.12 69.85 0)
 			(effects
@@
 			(project ""
 				(path "/0de7b960-2097-47c8-970c-7acab0ada146/6c5d3f5c-4c22-4772-8235-2f35636af7f3"
-					(reference "#PWR016")
+					(reference "#PWR013")
 					(unit 1)
 				)
@@
 		(dnp no)
 		(fields_autoplaced yes)
-		(property "Reference" "#PWR019"
+		(property "Reference" "#PWR015"
 			(at 71.12 101.6 0)
 			(effects
@@
 			(project "ABRARACOURCIX_main_board"
 				(path "/0de7b960-2097-47c8-970c-7acab0ada146/6c5d3f5c-4c22-4772-8235-2f35636af7f3"
-					(reference "#PWR019")
+					(reference "#PWR015")
 					(unit 1)
 				)
@@
 		(on_board yes)
 		(dnp no)
-		(property "Reference" "#J6"
+		(property "Reference" "#J2"
 			(at 37.465 125.73 0)
 			(effects
@@
 			(project "ABRARACOURCIX_main_board"
 				(path "/0de7b960-2097-47c8-970c-7acab0ada146/6c5d3f5c-4c22-4772-8235-2f35636af7f3"
-					(reference "#J6")
+					(reference "#J2")
 					(unit 1)
 				)
@@
 		(dnp no)
 		(fields_autoplaced yes)
-		(property "Reference" "#PWR015"
+		(property "Reference" "#PWR011"
 			(at 63.5 31.75 0)
 			(effects
@@
 			(project "ABRARACOURCIX_main_board"
 				(path "/0de7b960-2097-47c8-970c-7acab0ada146/6c5d3f5c-4c22-4772-8235-2f35636af7f3"
-					(reference "#PWR015")
+					(reference "#PWR011")
 					(unit 1)
 				)
@@
 		(dnp no)
 		(fields_autoplaced yes)
-		(property "Reference" "#PWR020"
+		(property "Reference" "#PWR016"
 			(at 71.12 107.95 0)
 			(effects
@@
 			(project "ABRARACOURCIX_main_board"
 				(path "/0de7b960-2097-47c8-970c-7acab0ada146/6c5d3f5c-4c22-4772-8235-2f35636af7f3"
-					(reference "#PWR020")
+					(reference "#PWR016")
 					(unit 1)
 				)
@@
 		(dnp no)
 		(fields_autoplaced yes)
-		(property "Reference" "#PWR024"
+		(property "Reference" "#PWR012"
 			(at 63.5 48.26 0)
 			(effects
@@
 			(project "ABRARACOURCIX_main_board"
 				(path "/0de7b960-2097-47c8-970c-7acab0ada146/6c5d3f5c-4c22-4772-8235-2f35636af7f3"
-					(reference "#PWR024")
+					(reference "#PWR012")
 					(unit 1)
 				)
@@
 		(dnp no)
 		(fields_autoplaced yes)
-		(property "Reference" "#R3"
+		(property "Reference" "#R1"
 			(at 72.39 139.6999 0)
 			(effects
@@
 			(project ""
 				(path "/0de7b960-2097-47c8-970c-7acab0ada146/6c5d3f5c-4c22-4772-8235-2f35636af7f3"
-					(reference "#R3")
+					(reference "#R1")
 					(unit 1)
 				)
@@
 		(dnp no)
 		(fields_autoplaced yes)
-		(property "Reference" "J5"
+		(property "Reference" "J1"
 			(at 54.61 34.29 0)
 			(effects
@@
 			(project "ABRARACOURCIX_main_board"
 				(path "/0de7b960-2097-47c8-970c-7acab0ada146/6c5d3f5c-4c22-4772-8235-2f35636af7f3"
-					(reference "J5")
+					(reference "J1")
 					(unit 1)
 				)
@@
 		(on_board yes)
 		(dnp no)
-		(property "Reference" "J4"
+		(property "Reference" "J2"
 			(at 52.07 106.426 0)
 			(effects
@@
 			(project "ABRARACOURCIX_main_board"
 				(path "/0de7b960-2097-47c8-970c-7acab0ada146/6c5d3f5c-4c22-4772-8235-2f35636af7f3"
-					(reference "J4")
+					(reference "J2")
 					(unit 1)
 				)
@@
 		(dnp no)
 		(fields_autoplaced yes)
-		(property "Reference" "#R4"
+		(property "Reference" "#R2"
 			(at 72.39 149.8599 0)
 			(effects
@@
 			(project ""
 				(path "/0de7b960-2097-47c8-970c-7acab0ada146/6c5d3f5c-4c22-4772-8235-2f35636af7f3"
-					(reference "#R4")
+					(reference "#R2")
 					(unit 1)
 				)
@@
 		(dnp no)
 		(fields_autoplaced yes)
-		(property "Reference" "#J4"
+		(property "Reference" "#J1"
 			(at 53.975 60.96 0)
 			(effects
@@
 			(project ""
 				(path "/0de7b960-2097-47c8-970c-7acab0ada146/6c5d3f5c-4c22-4772-8235-2f35636af7f3"
-					(reference "#J4")
-					(unit 1)
-				)
+					(reference "#J1")
+					(unit 1)
+				)
