File: ABRARACOURCIX_main_board-2025-11-06_181406/Output_interface.kicad_sch (KiCad schematic)
At the start: 12 parts, among them J10 Conn_01x03_Socket, J11 Conn_01x03_Socket, J6 Conn_01x03_Socket, J7 XT60PW-F, J8 Conn_01x03_Socket, J9 Conn_01x03_Socket, Q1 MMBT3904

Commit message: Modifs au circuit d'alim
Parts:
- J7: footprint XT60PW-F:AMASS_XT60PW-F -> Librairie_footprint:AMASS_XT60PW-F
Changed lines of the file:
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@@
 			)
 		)
-		(property "Footprint" "XT60PW-F:AMASS_XT60PW-F"
+		(property "Footprint" "Librairie_footprint:AMASS_XT60PW-F"
 			(at 81.28 148.59 0)
 			(effects

Commit message: Modif circuit d'arrêt
Parts:
- removed J7: XT60PW-F, Librairie_footprint:AMASS_XT60PW-F, symbol GAUL_ABRARACOURCIX:XT60PW-F
Other:
- note removed: "Output to ESC Max 30 A 15 V XT60 Female"

Commit message: Placement des composantes 95%
Parts:
- C27: footprint Capacitor_SMD:C_1206_3216Metric_Pad1.33x1.80mm_HandSolder -> Librairie_footprint:CAP_R533W520050P0K_KEM
Changed lines of the file:
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@@
 			)
 		)
-		(property "Footprint" "Capacitor_SMD:C_1206_3216Metric_Pad1.33x1.80mm_HandSolder"
+		(property "Footprint" "Librairie_footprint:CAP_R533W520050P0K_KEM"
 			(at 45.4152 85.09 0)
 			(effects

Commit message: Documentation de composantes
Parts:
- C27: footprint Librairie_footprint:CAP_R533W520050P0K_KEM -> Librairie_footprint:CAP_MU_15750_RUB-L
Other:
- moved on the sheet: J6
Changed lines of the file:
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@@
 	(rectangle
 		(start 36.83 137.16)
-		(end 116.84 177.8)
+		(end 105.41 156.21)
 		(stroke
 			(width 0)
@@
 	(text "Blanc\n\nNoir\n"
 		(exclude_from_sim no)
-		(at 78.232 166.624 0)
+		(at 76.962 143.764 0)
 		(effects
 			(font
@@
 	)
 	(no_connect
-		(at 69.85 166.37)
+		(at 68.58 143.51)
 	)
 	(wire
@@
 	(wire
 		(pts
-			(xy 67.31 163.83) (xy 69.85 163.83)
-		)
-		(stroke
-			(width 0)
-			(type default)
-		)
-	)
-	(wire
-		(pts
-			(xy 69.85 171.45) (xy 69.85 168.91)
+			(xy 66.04 140.97) (xy 68.58 140.97)
+		)
+		(stroke
+			(width 0)
+			(type default)
+		)
+	)
+	(wire
+		(pts
+			(xy 68.58 148.59) (xy 68.58 146.05)
 		)
 		(stroke
@@
 	(global_label "PWM_Moteur"
 		(shape input)
-		(at 67.31 163.83 180)
+		(at 66.04 140.97 180)
 		(fields_autoplaced yes)
 		(effects
@@
 		)
 		(property "Intersheetrefs" "${INTERSHEET_REFS}"
-			(at 52.8345 163.83 0)
+			(at 51.5645 140.97 0)
 			(effects
 				(font
@@
 	(symbol
 		(lib_id "Connector:Conn_01x03_Socket")
-		(at 74.93 166.37 0)
+		(at 73.66 143.51 0)
 		(unit 1)
 		(exclude_from_sim no)
@@
 		(dnp no)
 		(property "Reference" "J6"
-			(at 85.852 164.338 0)
+			(at 84.582 141.478 0)
 			(effects
 				(font
@@
 		)
 		(property "Value" "Conn_01x03_Socket"
-			(at 84.582 166.878 0)
+			(at 83.312 144.018 0)
 			(effects
 				(font
@@
 		)
 		(property "Footprint" "Connector_PinHeader_2.54mm:PinHeader_1x03_P2.54mm_Horizontal"
-			(at 74.93 166.37 0)
+			(at 73.66 143.51 0)
 			(effects
 				(font
@@
 		)
 		(property "Datasheet" "~"
-			(at 74.93 166.37 0)
+			(at 73.66 143.51 0)
 			(effects
 				(font
@@
 		)
 		(property "Description" "Generic connector, single row, 01x03, script generated"
-			(at 74.93 166.37 0)
+			(at 73.66 143.51 0)
 			(effects
 				(font
@@
 	(symbol
 		(lib_id "power:GND")
-		(at 69.85 171.45 0)
+		(at 68.58 148.59 0)
 		(unit 1)
 		(exclude_from_sim no)
@@
 		(fields_autoplaced yes)
 		(property "Reference" "#PWR046"
-			(at 69.85 177.8 0)
+			(at 68.58 154.94 0)
 			(effects
 				(font
@@
 		)
 		(property "Value" "GND"
-			(at 69.85 176.53 0)
+			(at 68.58 153.67 0)
 			(effects
 				(font
@@
 		)
 		(property "Footprint" ""
-			(at 69.85 171.45 0)
+			(at 68.58 148.59 0)
 			(effects
 				(font
@@
 		)
 		(property "Datasheet" ""
-			(at 69.85 171.45 0)
+			(at 68.58 148.59 0)
 			(effects
 				(font
@@
 		)
 		(property "Description" "Power symbol creates a global label with name \"GND\" , ground"
-			(at 69.85 171.45 0)
+			(at 68.58 148.59 0)
 			(effects
 				(font
@@
 			)
 		)
-		(property "Footprint" "Librairie_footprint:CAP_R533W520050P0K_KEM"
+		(property "Footprint" "Librairie_footprint:CAP_MU_15750_RUB-L"
 			(at 45.4152 85.09 0)
 			(effects

Commit message: Routing terminé (v1)
Parts:
- renumbered C27 to C11, J11 to J3, J9 to J4, J8 to J5, J10 to J6, J6 to J7
Changed lines of the file:
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@@
 		(on_board yes)
 		(dnp no)
-		(property "Reference" "J10"
+		(property "Reference" "J6"
 			(at 89.408 115.57 0)
 			(effects
@@
 			(project "ABRARACOURCIX_main_board"
 				(path "/0de7b960-2097-47c8-970c-7acab0ada146/f5120b67-a5cd-4c16-9638-751b3f9906f3"
-					(reference "J10")
+					(reference "J6")
 					(unit 1)
 				)
@@
 		(dnp no)
 		(fields_autoplaced yes)
-		(property "Reference" "#PWR027"
+		(property "Reference" "#PWR023"
 			(at 77.47 73.66 0)
 			(effects
@@
 			(project "ABRARACOURCIX_main_board"
 				(path "/0de7b960-2097-47c8-970c-7acab0ada146/f5120b67-a5cd-4c16-9638-751b3f9906f3"
-					(reference "#PWR027")
+					(reference "#PWR023")
 					(unit 1)
 				)
@@
 		(on_board yes)
 		(dnp no)
-		(property "Reference" "J6"
+		(property "Reference" "J7"
 			(at 84.582 141.478 0)
 			(effects
@@
 			(project ""
 				(path "/0de7b960-2097-47c8-970c-7acab0ada146/f5120b67-a5cd-4c16-9638-751b3f9906f3"
-					(reference "J6")
+					(reference "J7")
 					(unit 1)
 				)
@@
 		(dnp no)
 		(fields_autoplaced yes)
-		(property "Reference" "#PWR046"
+		(property "Reference" "#PWR032"
 			(at 68.58 154.94 0)
 			(effects
@@
 			(project "ABRARACOURCIX_main_board"
 				(path "/0de7b960-2097-47c8-970c-7acab0ada146/f5120b67-a5cd-4c16-9638-751b3f9906f3"
-					(reference "#PWR046")
+					(reference "#PWR032")
 					(unit 1)
 				)
@@
 		(dnp no)
 		(fields_autoplaced yes)
-		(property "Reference" "#PWR023"
+		(property "Reference" "#PWR030"
 			(at 77.47 124.46 0)
 			(effects
@@
 			(project ""
 				(path "/0de7b960-2097-47c8-970c-7acab0ada146/f5120b67-a5cd-4c16-9638-751b3f9906f3"
-					(reference "#PWR023")
+					(reference "#PWR030")
 					(unit 1)
 				)
@@
 		(dnp no)
 		(fields_autoplaced yes)
-		(property "Reference" "#PWR045"
+		(property "Reference" "#PWR025"
 			(at 44.45 81.28 0)
 			(effects
@@
 			(project "ABRARACOURCIX_main_board"
 				(path "/0de7b960-2097-47c8-970c-7acab0ada146/f5120b67-a5cd-4c16-9638-751b3f9906f3"
-					(reference "#PWR045")
+					(reference "#PWR025")
 					(unit 1)
 				)
@@
 		(dnp no)
 		(fields_autoplaced yes)
-		(property "Reference" "#PWR044"
+		(property "Reference" "#PWR026"
 			(at 44.45 91.44 0)
 			(effects
@@
 			(project "ABRARACOURCIX_main_board"
 				(path "/0de7b960-2097-47c8-970c-7acab0ada146/f5120b67-a5cd-4c16-9638-751b3f9906f3"
-					(reference "#PWR044")
+					(reference "#PWR026")
 					(unit 1)
 				)
@@
 		(on_board yes)
 		(dnp no)
-		(property "Reference" "J8"
+		(property "Reference" "J5"
 			(at 89.408 90.17 0)
 			(effects
@@
 			(project "ABRARACOURCIX_main_board"
 				(path "/0de7b960-2097-47c8-970c-7acab0ada146/f5120b67-a5cd-4c16-9638-751b3f9906f3"
-					(reference "J8")
+					(reference "J5")
 					(unit 1)
 				)
@@
 		(dnp no)
 		(fields_autoplaced yes)
-		(property "Reference" "#PWR028"
+		(property "Reference" "#PWR024"
 			(at 77.47 78.74 0)
 			(effects
@@
 			(project "ABRARACOURCIX_main_board"
 				(path "/0de7b960-2097-47c8-970c-7acab0ada146/f5120b67-a5cd-4c16-9638-751b3f9906f3"
-					(reference "#PWR028")
+					(reference "#PWR024")
 					(unit 1)
 				)
@@
 		(dnp yes)
 		(fields_autoplaced yes)
-		(property "Reference" "#PWR011"
+		(property "Reference" "#PWR022"
 			(at 231.14 53.34 0)
 			(effects
@@
 			(project "ABRARACOURCIX_main_board"
 				(path "/0de7b960-2097-47c8-970c-7acab0ada146/f5120b67-a5cd-4c16-9638-751b3f9906f3"
-					(reference "#PWR011")
+					(reference "#PWR022")
 					(unit 1)
 				)
@@
 		(dnp no)
 		(fields_autoplaced yes)
-		(property "Reference" "#PWR022"
+		(property "Reference" "#PWR031"
 			(at 77.47 129.54 0)
 			(effects
@@
 			(project "ABRARACOURCIX_main_board"
 				(path "/0de7b960-2097-47c8-970c-7acab0ada146/f5120b67-a5cd-4c16-9638-751b3f9906f3"
-					(reference "#PWR022")
+					(reference "#PWR031")
 					(unit 1)
 				)
@@
 		(on_board yes)
 		(dnp no)
-		(property "Reference" "J11"
+		(property "Reference" "J3"
 			(at 89.408 40.64 0)
 			(effects
@@
 			(project "ABRARACOURCIX_main_board"
 				(path "/0de7b960-2097-47c8-970c-7acab0ada146/f5120b67-a5cd-4c16-9638-751b3f9906f3"
-					(reference "J11")
+					(reference "J3")
 					(unit 1)
 				)
@@
 		(on_board no)
 		(dnp yes)
-		(property "Reference" "#PWR074"
+		(property "Reference" "#PWR027"
 			(at 231.14 95.25 0)
 			(effects
@@
 			(project "ABRARACOURCIX_main_board"
 				(path "/0de7b960-2097-47c8-970c-7acab0ada146/f5120b67-a5cd-4c16-9638-751b3f9906f3"
-					(reference "#PWR074")
+					(reference "#PWR027")
 					(unit 1)
 				)
@@
 		(on_board yes)
 		(dnp no)
-		(property "Reference" "J9"
+		(property "Reference" "J4"
 			(at 89.408 64.77 0)
 			(effects
@@
 			(project "ABRARACOURCIX_main_board"
 				(path "/0de7b960-2097-47c8-970c-7acab0ada146/f5120b67-a5cd-4c16-9638-751b3f9906f3"
-					(reference "J9")
+					(reference "J4")
 					(unit 1)
 				)
@@
 		(dnp no)
 		(fields_autoplaced yes)
-		(property "Reference" "#PWR030"
+		(property "Reference" "#PWR021"
 			(at 77.47 54.61 0)
 			(effects
@@
 			(project "ABRARACOURCIX_main_board"
 				(path "/0de7b960-2097-47c8-970c-7acab0ada146/f5120b67-a5cd-4c16-9638-751b3f9906f3"
-					(reference "#PWR030")
+					(reference "#PWR021")
 					(unit 1)
 				)
@@
 		(dnp no)
 		(fields_autoplaced yes)
-		(property "Reference" "C27"
+		(property "Reference" "C11"
 			(at 48.26 80.0099 0)
 			(effects
@@
 			(project ""
 				(path "/0de7b960-2097-47c8-970c-7acab0ada146/f5120b67-a5cd-4c16-9638-751b3f9906f3"
-					(reference "C27")
+					(reference "C11")
 					(unit 1)
 				)
@@
 		(dnp no)
 		(fields_autoplaced yes)
-		(property "Reference" "#PWR025"
+		(property "Reference" "#PWR028"
 			(at 77.47 99.06 0)
 			(effects
@@
 			(project "ABRARACOURCIX_main_board"
 				(path "/0de7b960-2097-47c8-970c-7acab0ada146/f5120b67-a5cd-4c16-9638-751b3f9906f3"
-					(reference "#PWR025")
+					(reference "#PWR028")
 					(unit 1)
 				)
@@
 		(dnp no)
 		(fields_autoplaced yes)
-		(property "Reference" "#PWR029"
+		(property "Reference" "#PWR020"
 			(at 77.47 49.53 0)
 			(effects
@@
 			(project "ABRARACOURCIX_main_board"
 				(path "/0de7b960-2097-47c8-970c-7acab0ada146/f5120b67-a5cd-4c16-9638-751b3f9906f3"
-					(reference "#PWR029")
+					(reference "#PWR020")
 					(unit 1)
 				)
@@
 		(dnp no)
 		(fields_autoplaced yes)
-		(property "Reference" "#PWR026"
+		(property "Reference" "#PWR029"
 			(at 77.47 104.14 0)
 			(effects
@@
 			(project "ABRARACOURCIX_main_board"
 				(path "/0de7b960-2097-47c8-970c-7acab0ada146/f5120b67-a5cd-4c16-9638-751b3f9906f3"
-					(reference "#PWR026")
-					(unit 1)
-				)
+					(reference "#PWR029")
+					(unit 1)
+				)
